File: FrontEndPrototype_Rev1/ABBCore_alt.kicad_sch (KiCad schematic)
At the start: 26 parts, among them J11 Conn_02x04_Odd_Even, J12 Conn_02x02_Odd_Even, SW1 MAX4704, U1 ADA4807-2ACP, U9 74LVC1G139

Commit message: Checking if Branch Updates Work
Parts:
- gave numbers to parts that had none: 21
- renumbered U1 to U2

Commit message: Small Updates
Parts:
- removed C9: 1u, Capacitor_SMD:C_0603_1608Metric_Pad1.08x0.95mm_HandSolder, symbol Device:C_Small
- removed Cb13: 0.1u, Capacitor_SMD:C_0603_1608Metric_Pad1.08x0.95mm_HandSolder, symbol Device:C_Small
- removed J11: Conn_02x04_Odd_Even, Connector_PinHeader_2.54mm:PinHeader_2x04_P2.54mm_Vertical_SMD, symbol Connector_Generic:Conn_02x04_Odd_Even
- removed J12: Conn_02x02_Odd_Even, Connector_PinHeader_2.54mm:PinHeader_1x04_P2.54mm_Vertical_SMD_Pin1Right, symbol Connector_Generic:Conn_01x04
- removed R10: 100, Resistor_SMD:R_0603_1608Metric_Pad0.98x0.95mm_HandSolder, symbol Device:R_Small_US
- removed SW1: MAX4704, Package_DFN_QFN:DFN-12-1EP_3x3mm_P0.5mm_EP1.6x2.5mm, symbol FrontEndPrototype_Rev1-rescue:MAX4704
- removed U9: 74LVC1G139, Package_SO:VSSOP-8_2.3x2mm_P0.5mm, symbol 74xGxx:74LVC1G139
- added U1: CD74AC238, Package_SO:TSSOP-16_4.4x5mm_P0.65mm, symbol 74xx:CD74AC238
- Cb14: value 1u -> 0.1u
- Rf3: value 50k -> 39k
Connections:
- net D0: now also U1.1 (A0)
- net D1: now also U1.2 (A1)
- net GND: now also U1.3 (A2), U1.4 (~{E1}), U1.5 (~{E2}), U1.8 (GND)
- net Vdd: now also U1.16 (VCC), U1.6 (E3)
- net ~{TIA1_SHDN}: now also U1.15 (Y0)
- net ~{TIA2_SHDN}: now also U1.14 (Y1)
- net ~{TIA3_SHDN}: now also U1.13 (Y2)
- net ~{TIA4_SHDN}: now also U1.12 (Y3)
- no-connect marks 1 -> 4
Other:
- note removed: "High Isolation Low Cross-Talk Multiplexer (Use Jumpers and EN to route around)"
