File: FrontEndPrototype_Rev1/MCU_Connections_STM32WB55.kicad_sch (KiCad schematic)
At the start: 2 parts, among them J1 Conn_02x19_Odd_Even, J2 Conn_02x19_Odd_Even

Commit message: Small Updates
Connections:
- net PA5: now reaches J2.11 (Pin_11)
- net QSPI_IO0: no longer names the net of J2.5 (Pin_5)
- net QSPI_IO1: no longer names the net of J2.3 (Pin_3)
- net QSPI_IO2 renamed PA7
- net QSPI_IO3 renamed PA6
- net QSPI_SCK renamed PA4
- net Tim2_PWM_2 renamed PA2
- net Tim2_PWM_3 renamed PA3
Changed lines of the file:
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@@
+	(wire
+		(pts
+			(xy 102.87 57.15) (xy 105.41 57.15)
+		)
+		(stroke
+			(width 0)
+			(type default)
+		)
+	)
 	(wire
 		(pts
@@
 		)
 	)
-	(hierarchical_label "QSPI_IO1"
-		(shape output)
-		(at 102.87 46.99 180)
-		(fields_autoplaced yes)
-		(effects
-			(font
-				(size 1.27 1.27)
-			)
-			(justify right)
-		)
-	)
 	(hierarchical_label "PC12"
 		(shape output)
@@
 		)
 	)
+	(hierarchical_label "PA5"
+		(shape output)
+		(at 102.87 57.15 180)
+		(fields_autoplaced yes)
+		(effects
+			(font
+				(size 1.27 1.27)
+			)
+			(justify right)
+		)
+	)
 	(hierarchical_label "PA1"
 		(shape output)
@@
 		)
 	)
-	(hierarchical_label "QSPI_IO2"
+	(hierarchical_label "PA7"
 		(shape output)
 		(at 102.87 62.23 180)
@@
 		)
 	)
-	(hierarchical_label "QSPI_SCK"
+	(hierarchical_label "PA4"
 		(shape output)
 		(at 102.87 64.77 180)
@@
 		)
 	)
-	(hierarchical_label "QSPI_IO0"
-		(shape output)
-		(at 102.87 49.53 180)
-		(fields_autoplaced yes)
-		(effects
-			(font
-				(size 1.27 1.27)
-			)
-			(justify right)
-		)
-	)
 	(hierarchical_label "Vdd"
 		(shape output)
@@
 		)
 	)
-	(hierarchical_label "Tim2_PWM_2"
+	(hierarchical_label "PA2"
 		(shape output)
 		(at 102.87 87.63 180)
@@
 		)
 	)
-	(hierarchical_label "Tim2_PWM_3"
+	(hierarchical_label "PA3"
 		(shape output)
 		(at 102.87 90.17 180)
@@
 		)
 	)
-	(hierarchical_label "QSPI_IO3"
+	(hierarchical_label "PA6"
 		(shape output)
 		(at 102.87 59.69 180)
