File: Power_Management_Board/Power_Management_Board.kicad_sch (KiCad schematic)
At the start: 31 parts, among them J1 USB_C_Receptacle_PowerOnly_6P, J2 Screw_Terminal_01x02, J3 Conn_02x19_Odd_Even, J4 Conn_02x19_Odd_Even, Q1 PMOS, U1 LD39200, U2 LD39050, U3 MCP73831-2-OT

Commit message: Finished USB-C Power Board Design
Parts:
- removed J2: Screw_Terminal_01x02, symbol Connector:Screw_Terminal_01x02
- removed Q1: PMOS, symbol Simulation_SPICE:PMOS
- added C12, C13, C16: 1uF, Capacitor_SMD:C_0603_1608Metric_Pad1.08x0.95mm_HandSolder, symbol Device:C_Small
- added C14, C15: 10uF, Capacitor_SMD:C_0603_1608Metric_Pad1.08x0.95mm_HandSolder, symbol Device:C_Small
- added J2: B2PS-VH, Connector_JST:JST_VH_B2PS-VH_1x02_P3.96mm_Horizontal, symbol Connector:Conn_01x02_Socket
- added Q1: SSM3J358R, Package_TO_SOT_SMD:SOT-23-3, symbol FrontEndPrototype_Rev1-rescue:SSM3J358R
- added R10, R11: 10k, Resistor_SMD:R_0603_1608Metric_Pad0.98x0.95mm_HandSolder, symbol Device:R_Small_US
- added U5: ADR4530, Package_SO:SOIC-8_3.9x4.9mm_P1.27mm, symbol Reference_Voltage:ADR4530
- added U6: ADA4807-2ACP, Package_CSP:LFCSP-WD-10-1EP_3x3mm_P0.5mm_EP1.64x2.38mm, symbol Amplifier_Operational:ADA4807-2ACP
- added U7: ADP7118-1.8, Package_TO_SOT_SMD:TSOT-23-5, symbol Regulator_Linear:ADP7142AUJZ-1.8
- C1, C2, C3, C4, C5, C6, C7, C8, C9: footprint (none) -> Capacitor_SMD:C_0603_1608Metric_Pad1.08x0.95mm_HandSolder
- D1: value D -> MSS1P3L; footprint (none) -> Diode_SMD:D_MicroSMP_AK
- J1: footprint (none) -> Connector_USB:USB_C_Receptacle_GCT_USB4125-xx-x_6P_TopMnt_Horizontal
- J3, J4: footprint (none) -> Connector_PinHeader_2.54mm:PinHeader_2x19_P2.54mm_Vertical
- R1, R2, R3, R4, R5, R6, R7, R8, R9: footprint (none) -> Resistor_SMD:R_0603_1608Metric_Pad0.98x0.95mm_HandSolder
- SW1: value ~ -> Rocker Switch SPST; footprint (none) -> Connector_PinHeader_2.54mm:PinHeader_1x02_P2.54mm_Vertical
Connections:
- net 5V_USB: now also Q1.1 (G)
- net GND: now also J3.19 (Pin_19), J3.20 (Pin_20), J3.8 (Pin_8), J4.20 (Pin_20), J4.32 (Pin_32), J4.38 (Pin_38), J4.9 (Pin_9), C12.2, C13.1, C14.2, C15.2, C16.2, J2.2 (Pin_2), R11.2, U5.4 (GND), U6.11 (EPAD), U6.4 (V-), U7.2 (GND)
- net V_BATT: now also J2.1 (Pin_1), Q1.3 (D)
- net Vdd_Heater: now also J3.37 (Pin_37)
- net Vdd_Main: now also J3.5 (Pin_5), C12.1, C14.1, C15.1, C16.1, U5.2 (IN), U6.10 (V+), U7.1 (VIN), U7.4 (SENSE/ADJ), U7.5 (VOUT)
- net V_IN: now reaches D1.1 (K), SW1.1 (A)
- net V_IN: now also C1.1, C6.1, C7.2, U1.7 (Vin), U1.8 (Vin), U2.6 (Vin), Q1.2 (S)
- net ~{SHDN_IA}: now reaches J4.4 (Pin_4)
- net ~{SHDN_IA}: now also U6.5 (~{DISABLE1}), U6.6 (~{DISABLE2}), U7.3 (EN)
- new net: SW1.2 (B), U1.6 (EN), U2.1 (EN)
- new net: C13.2, U5.6 (OUT), U6.3 (+)
- new net: R10.2, R11.1, U6.7 (+)
- new net ADC_VREF: R10.1, U6.1, U6.2 (-)
- new net Vmid: U6.8 (-), U6.9
Other:
- note added: "- Rds_On should be very low to avoid excess power drain from battery - Continuous drain current must go up to 1A"
- note added: "Heater GND should connect to main system GND near input of power cable"
- note added: "Main Power Switch Enables LDOs when on"
- note added: "Reference Generation Vref = 3.0 V Vmid = 1.5 V"
- note removed: "Main Power Switch"
- company: (none) -> BioMicrosystems Laboratory
- title: (none) -> Gen II Power Board
- moved on the sheet: C1, J3
