File: MeasurementBoard_Rev2/ABBCore_alt.kicad_sch (KiCad schematic)
At the start: 20 parts, among them J10 MIllMaxSpringConnector, J3 MIllMaxSpringConnector, J4 MIllMaxSpringConnector, J5 MIllMaxSpringConnector, J6 MIllMaxSpringConnector, J7 MIllMaxSpringConnector, J8 MIllMaxSpringConnector, J9 MIllMaxSpringConnector, U1 CD74AC238, U2 ADA4807-2ACP

Commit message: Finished Measurement Board Update Minus Heater Board Connections
Parts:
- removed Cb14: 0.1u, Capacitor_SMD:C_0603_1608Metric_Pad1.08x0.95mm_HandSolder, symbol Device:C_Small
- removed U1: CD74AC238, Package_SO:TSSOP-16_4.4x5mm_P0.65mm, symbol 74xx:CD74AC238
- renumbered J6 to J1, J4 to J2, J5 to J3, J3 to J4, J7 to J5, J8 to J6, J9 to J7, J10 to J8
Connections:
- net CCOut_1: now also J6.1; no longer J1.1
- net CCOut_2: now also J5.1; no longer J7.1
- net CCOut_4: now also J1.1; no longer J8.1
- net V_Drive: now also J7.1, J8.1; no longer J5.1, J6.1
- no-connect marks 4 -> 0
Other:
- note removed: "Decoder for multiplexing"
- moved on the sheet: J1, J3, J4, J5, J6, J7, J8
