File: MeasurementBoard_Rev2/ADC_Drivers_4807_pseudo.kicad_sch (KiCad schematic)
At the start: 15 parts, among them U6 ADA4807-2ACP, U7 AD4002_LFSCP-10, U8 AD4002_LFSCP-10

Commit message: Final commit before order
Parts:
- U8: footprint footprints:CP_10_9_ADI -> Package_CSP:LFCSP-WD-10-1EP_3x3mm_P0.5mm_EP1.64x2.38mm
Changed lines of the file:
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@@
 			)
 		)
-		(property "Footprint" "footprints:CP_10_9_ADI"
+		(property "Footprint" "Package_CSP:LFCSP-WD-10-1EP_3x3mm_P0.5mm_EP1.64x2.38mm"
 			(at 180.34 38.1 0)
 			(effects
