File: MeasurementBoard_Rev2/CC_Driver.kicad_sch (KiCad schematic)
At the start: 12 parts, among them U2 ADA4807-2ACP

Commit message: Final commit before order
Parts:
- RT1: value 0 -> NC
Changed lines of the file:
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@@
 			)
 		)
-		(property "Value" "0"
+		(property "Value" "NC"
 			(at 33.9344 57.15 90)
 			(effects
