File: Raspi_Zero_TFT_Interface/Raspi_Zero_TFT_Interface.kicad_sch (KiCad schematic)
At the start: 14 parts, among them CN1 USB_C_Receptacle_PowerOnly_6P, CN2 B2PS-VH, CN3 Molex FPC 541044031, CN4 Molex FPC 52271-0679, CN5 Conn_02x20_Odd_Even, CN6 Molex FPC 52271-0679, U1 AP5725WG-7

Commit message: First draft layout of power pi board
Parts:
- CN2: value B2PS-VH -> B2B-XH-A; footprint Connector_JST:JST_VH_B2P-VH_1x02_P3.96mm_Vertical -> Connector_JST:JST_XH_B2B-XH-A_1x02_P2.50mm_Vertical
- CN5: footprint Connector_Samtec_HLE_SMD:Samtec_HLE-120-02-xxx-DV-BE_2x20_P2.54mm_Horizontal -> Connector_PinHeader_2.54mm:PinHeader_2x20_P2.54mm_Vertical
Connections:
- net B1: now also CN5.30 (Pin_30); no longer CN5.29 (Pin_29)
- net B2: now also CN5.32 (Pin_32); no longer CN5.31 (Pin_31)
- net B3: now also CN5.25 (Pin_25); no longer CN5.26 (Pin_26)
- net B4: now also CN5.23 (Pin_23); no longer CN5.24 (Pin_24)
- net B5: now also CN5.22 (Pin_22); no longer CN5.21 (Pin_21)
- net B6: now also CN5.20 (Pin_20); no longer CN5.19 (Pin_19)
- net B7: now also CN5.24 (Pin_24); no longer CN5.23 (Pin_23)
- net CLK: now also CN5.28 (Pin_28); no longer CN5.27 (Pin_27)
- net DE: now also CN5.27 (Pin_27); no longer CN5.28 (Pin_28)
- net DISP: now also CN5.37 (Pin_37); no longer CN5.38 (Pin_38)
- net G0: no longer CN5.32 (Pin_32)
- net G1: now also CN5.34 (Pin_34); no longer CN5.33 (Pin_33)
- net G2: now also CN5.16 (Pin_16); no longer CN5.15 (Pin_15)
- net G3: now also CN5.15 (Pin_15); no longer CN5.16 (Pin_16)
- net G4: now also CN5.35 (Pin_35); no longer CN5.36 (Pin_36)
- net G5: now also CN5.12 (Pin_12); no longer CN5.11 (Pin_11)
- net G6: now also CN5.11 (Pin_11); no longer CN5.12 (Pin_12)
- net G7: now also CN5.36 (Pin_36); no longer CN5.35 (Pin_35)
- net GND: now also CN5.10 (Pin_10), CN5.13 (Pin_13), CN5.19 (Pin_19), CN5.26 (Pin_26), CN5.29 (Pin_29), CN5.33 (Pin_33), CN5.40 (Pin_40), CN5.5 (Pin_5); no longer CN5.14 (Pin_14), CN5.20 (Pin_20), CN5.25 (Pin_25), CN5.30 (Pin_30), CN5.34 (Pin_34), CN5.39 (Pin_39), CN5.6 (Pin_6), CN5.9 (Pin_9)
- net PWM_EN: now also CN5.31 (Pin_31)
- net Vcc: now also CN5.1 (Pin_1), CN5.3 (Pin_3); no longer CN5.2 (Pin_2), CN5.4 (Pin_4)
- net 3V3 renamed 3V3_Pi
- net 3V3_Pi: now also CN5.18 (Pin_18), CN5.2 (Pin_2); no longer CN5.1 (Pin_1), CN5.17 (Pin_17), CN6.6
- net GPIO14 renamed UART_TX
- net UART_TX: now also CN5.7 (Pin_7); no longer CN5.8 (Pin_8)
- net GPIO15 renamed UART_RX
- net UART_RX: now also CN5.9 (Pin_9); no longer CN5.10 (Pin_10)
- net GPIO2 renamed SDA
- net SDA: now also CN5.4 (Pin_4); no longer CN5.3 (Pin_3)
- net GPIO21 renamed R1
- net R1: now also CN5.39 (Pin_39); no longer CN5.40 (Pin_40)
- net GPIO24 renamed R4
- net R4: now also CN5.17 (Pin_17); no longer CN5.18 (Pin_18)
- net GPIO25 renamed R5
- net R5: now also CN5.21 (Pin_21); no longer CN5.22 (Pin_22)
- net GPIO26 renamed R6
- net R6: now also CN5.38 (Pin_38); no longer CN5.37 (Pin_37)
- net GPIO27 renamed R7
- net R7: now also CN5.14 (Pin_14); no longer CN5.13 (Pin_13)
- net GPIO3 renamed SCL
- net SCL: now also CN5.6 (Pin_6); no longer CN5.5 (Pin_5)
- net GPIO4 renamed ~{INT}
- net ~{INT}: now also CN5.8 (Pin_8); no longer CN5.7 (Pin_7)
- new net 3V3_Main: CN6.6
- no-connect marks 10 -> 11
Other:
- note added: "Raspberry Pi Zero 2W Connector. Right and left sides are flipped for bottom facing connector"
- note removed: "Raspberry Pi Zero 2W Connector"

Commit message: Completed (unflipped) board
Other:
- note added: "USB_VCC 1 and 2 should be monitored by MCU ADC channels to determine how much current source can supply. If too low, MCU should not allow certain functions and warn the user."
- note removed: "Optional Current Source Capability Monitoring"
Changed lines of the file:
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@@
-		)
-	)
-	(text "Optional Current Source\nCapability Monitoring"
-		(exclude_from_sim no)
-		(at 229.616 146.812 0)
-		(effects
-			(font
-				(size 1.27 1.27)
-			)
 		)
 	)
@@
 		)
 	)
+	(text "USB_VCC 1 and 2 should be monitored by MCU \nADC channels to determine how much current \nsource can supply. If too low, MCU should not\nallow certain functions and warn the user. "
+		(exclude_from_sim no)
+		(at 206.502 158.75 0)
+		(effects
+			(font
+				(size 1.27 1.27)
+			)
+			(justify left bottom)
+		)
+	)

Commit message: Partial Update
Connections:
- net 3V3_Pi: now also CN3.39; no longer CN3.4
- net B0: now also CN3.22; no longer CN3.21
- net B1: now also CN3.21; no longer CN3.22
- net B2: now also CN3.20; no longer CN3.23
- net B3: now also CN3.19; no longer CN3.24
- net B4: now also CN3.18; no longer CN3.25
- net B5: now also CN3.17; no longer CN3.26
- net B6: now also CN3.16; no longer CN3.27
- net B7: now also CN3.15; no longer CN3.28
- net CLK: now also CN3.13; no longer CN3.30
- net DE: now also CN3.9; no longer CN3.34
- net DISP: now also CN3.12; no longer CN3.31
- net G0: now also CN3.30; no longer CN3.13
- net G1: now also CN3.29; no longer CN3.14
- net G2: now also CN3.28, CN3.36; no longer CN3.15, CN3.7
- net G3: now also CN3.27, CN3.35; no longer CN3.16, CN3.8
- net G4: now also CN3.26; no longer CN3.17
- net G5: now also CN3.25; no longer CN3.18
- net G6: now also CN3.24; no longer CN3.19
- net G7: now also CN3.23; no longer CN3.20
- net GND: now also CN3.10, CN3.11, CN3.14, CN3.40, CN3.7, CN4.5; no longer CN3.29, CN3.3, CN3.32, CN3.33, CN3.36, CN4.2
- net LED+: now also CN3.P1; no longer CN3.2
- net LED-: now also CN3.P2; no longer CN3.1
- net R0: now also CN3.38; no longer CN3.5
- net R1: now also CN3.37; no longer CN3.6
- net R4: now also CN3.34; no longer CN3.9
- net R5: now also CN3.33; no longer CN3.10
- net R6: now also CN3.32; no longer CN3.11
- net R7: now also CN3.31; no longer CN3.12
- net SCL: now also CN4.4; no longer CN4.3
- net SDA: now also CN4.3; no longer CN4.4
- net ~{INT}: now also CN4.2; no longer CN4.5
Other:
- moved on the sheet: CN3

Commit message: Finalized Ras_Pi Power Board
Parts:
- added C1: 1uF, Capacitor_SMD:C_0603_1608Metric_Pad1.08x0.95mm_HandSolder, symbol Device:C_Small
Connections:
- net 3V3_Pi: now also CN3.37; no longer CN3.39
- net B0: now also CN3.20; no longer CN3.22
- net B1: now also CN3.19; no longer CN3.21
- net B2: now also CN3.18; no longer CN3.20
- net B3: now also CN3.17; no longer CN3.19
- net B4: now also CN3.16; no longer CN3.18
- net B5: now also CN3.15; no longer CN3.17
- net B6: now also CN3.14; no longer CN3.16
- net B7: now also CN3.13; no longer CN3.15
- net CLK: now also CN3.11; no longer CN3.13
- net DE: now also CN3.7; no longer CN3.9
- net DISP: now also CN3.10; no longer CN3.12
- net G0: now also CN3.28; no longer CN3.30
- net G1: now also CN3.27; no longer CN3.29
- net G2: now also CN3.26, CN3.34; no longer CN3.28, CN3.36
- net G3: now also CN3.25, CN3.33; no longer CN3.27, CN3.35
- net G4: now also CN3.24; no longer CN3.26
- net G5: now also CN3.23; no longer CN3.25
- net G6: now also CN3.22; no longer CN3.24
- net G7: now also CN3.21; no longer CN3.23
- net GND: now also CN3.12, CN3.38, CN3.5, CN3.8, CN3.9, C1.1; no longer CN3.10, CN3.11, CN3.14, CN3.40, CN3.7
- net LED+: now also CN3.39, C1.2; no longer CN3.P1
- net LED-: now also CN3.40; no longer CN3.P2
- net R0: now also CN3.36; no longer CN3.38
- net R1: now also CN3.35; no longer CN3.37
- net R4: now also CN3.32; no longer CN3.34
- net R5: now also CN3.31; no longer CN3.33
- net R6: now also CN3.30; no longer CN3.32
- net R7: now also CN3.29; no longer CN3.31

Commit message: Nearly Finalized Boards
Parts:
- removed CN6: Molex FPC 52271-0679, GenIILibrary:MOLEX_52271-0679, symbol 52271-0679:52271-0679
- added J1: 522070860, GenIILibrary:CON_522070860_MOL, symbol 2024-10-22_14-40-48:522070860
Connections:
- net Power_Management_Minimal/V_Batt+ is gone; now on net Power_Management_Minimal/V_Batt-: CN2.1 (Pin_1)
- net 3V3_Main: now also J1.6
- net GND: now also J1.2, J1.5
- net Power_Management_Minimal/V_Batt-: no longer CN2.2 (Pin_2)
- net UART_RX: now also J1.4
- net UART_TX: now also J1.3
- net Vcc: now also J1.1
- new net V_Batt: CN2.2 (Pin_2), J1.8
- new net ~{CHARGE_EN}: J1.7
- no-connect marks 11 -> 13
Other:
- sheet Power_Management_Minimal ports: added ~{CHARGE_EN}; removed none
- moved on the sheet: CN2
Changed lines of the file:
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@@
 		(color 0 0 0 0)
 	)
+	(junction
+		(at 223.52 129.54)
+		(diameter 0)
+		(color 0 0 0 0)
+	)
 	(no_connect
 		(at 35.56 83.82)
@@
 	)
 	(no_connect
+		(at 233.68 68.58)
+	)
+	(no_connect
 		(at 43.18 124.46)
 	)
 	(no_connect
+		(at 233.68 66.04)
+	)
+	(no_connect
 		(at 43.18 127)
 	)
@@
 	(wire
 		(pts
+			(xy 233.68 60.96) (xy 236.22 60.96)
+		)
+		(stroke
+			(width 0)
+			(type default)
+		)
+	)
+	(wire
+		(pts
 			(xy 246.38 121.92) (xy 246.38 123.19)
 		)
@@
 	(wire
 		(pts
-			(xy 219.71 132.08) (xy 222.25 132.08)
+			(xy 219.71 132.08) (xy 224.79 132.08)
 		)
 		(stroke
@@
 	(wire
 		(pts
+			(xy 180.34 129.54) (xy 193.04 129.54)
+		)
+		(stroke
+			(width 0)
+			(type default)
+		)
+	)
+	(wire
+		(pts
 			(xy 35.56 109.22) (xy 43.18 109.22)
 		)
@@
 	(wire
 		(pts
-			(xy 222.25 129.54) (xy 220.98 129.54)
+			(xy 224.79 129.54) (xy 223.52 129.54)
 		)
 		(stroke
@@
 	(wire
 		(pts
+			(xy 227.33 127) (xy 223.52 127)
+		)
+		(stroke
+			(width 0)
+			(type default)
+		)
+	)
+	(wire
+		(pts
 			(xy 246.38 128.27) (xy 246.38 130.81)
 		)
@@
 	(wire
 		(pts
+			(xy 233.68 63.5) (xy 241.3 63.5)
+		)
+		(stroke
+			(width 0)
+			(type default)
+		)
+	)
+	(wire
+		(pts
 			(xy 246.38 140.97) (xy 246.38 142.24)
 		)
@@
 	(wire
 		(pts
+			(xy 223.52 129.54) (xy 220.98 129.54)
+		)
+		(stroke
+			(width 0)
+			(type default)
+		)
+	)
+	(wire
+		(pts
 			(xy 87.63 35.56) (xy 102.87 35.56)
 		)
@@
 	(wire
 		(pts
+			(xy 223.52 127) (xy 223.52 129.54)
+		)
+		(stroke
+			(width 0)
+			(type default)
+		)
+	)
+	(wire
+		(pts
 			(xy 154.94 43.18) (xy 137.16 43.18)
 		)
@@
 		)
 	)
+	(label "~{CHARGE_EN}"
+		(at 180.34 129.54 0)
+		(fields_autoplaced yes)
+		(effects
+			(font
+				(size 1.27 1.27)
+			)
+			(justify left bottom)
+		)
+	)
 	(label "B1"
 		(at 35.56 86.36 0)
@@
 		)
 	)
+	(label "V_Batt"
+		(at 241.3 63.5 180)
+		(fields_autoplaced yes)
+		(effects
+			(font
+				(size 1.27 1.27)
+			)
+			(justify right bottom)
+		)
+	)
 	(label "R1"
 		(at 35.56 45.72 0)
@@
 		)
 	)
+	(label "~{CHARGE_EN}"
+		(at 236.22 60.96 0)
+		(fields_autoplaced yes)
+		(effects
+			(font
+				(size 1.27 1.27)
+			)
+			(justify left bottom)
+		)
+	)
 	(label "UART_RX"
 		(at 237.49 53.34 0)
@@
 		)
 	)
+	(label "V_Batt"
+		(at 227.33 127 180)
+		(fields_autoplaced yes)
+		(effects
+			(font
+				(size 1.27 1.27)
+			)
+			(justify right bottom)
+		)
+	)
 	(label "R0"
 		(at 35.56 43.18 0)
@@
 	(symbol
 		(lib_id "Connector:Conn_01x02_Socket")
-		(at 227.33 129.54 0)
+		(at 229.87 132.08 0)
+		(mirror x)
 		(unit 1)
 		(exclude_from_sim no)
@@
 		(dnp no)
 		(property "Reference" "CN2"
-			(at 226.695 124.46 0)
+			(at 227.965 139.954 0)
 			(effects
 				(font
@@
 		)
 		(property "Value" "B2B-XH-A"
-			(at 227.33 126.746 0)
+			(at 228.6 137.668 0)
 			(effects
 				(font
@@
 		)
 		(property "Footprint" "Connector_JST:JST_XH_B2B-XH-A_1x02_P2.50mm_Vertical"
-			(at 227.33 129.54 0)
+			(at 229.87 132.08 0)
 			(effects
 				(font
@@
 		)
 		(property "Datasheet" "~"
-			(at 227.33 129.54 0)
+			(at 229.87 132.08 0)
 			(effects
 				(font
@@
 		)
 		(property "Description" "Generic connector, single row, 01x02, script generated"
-			(at 227.33 129.54 0)
+			(at 229.87 132.08 0)
 			(effects
 				(font
@@
 	)
 	(symbol
-		(lib_id "52271-0679:52271-0679")
-		(at 226.06 50.8 0)
-		(unit 1)
-		(exclude_from_sim no)
-		(in_bom yes)
-		(on_board yes)
-		(dnp no)
-		(property "Reference" "CN6"
-			(at 226.06 36.322 0)
-			(effects
-				(font
-					(size 1.27 1.27)
-				)
-			)
-		)
-		(property "Value" "Molex FPC 52271-0679"
-			(at 226.06 38.862 0)
-			(effects
-				(font
-					(size 1.27 1.27)
-				)
-			)
-		)
-		(property "Footprint" "GenIILibrary:MOLEX_52271-0679"
-			(at 226.06 50.8 0)
-			(effects
-				(font
-					(size 1.27 1.27)
-				)
-				(justify bottom)
-				(hide yes)
-			)
-		)
-		(property "Datasheet" ""
-			(at 226.06 50.8 0)
-			(effects
-				(font
-					(size 1.27 1.27)
-				)
-				(hide yes)
-			)
-		)
-		(property "Description" ""
-			(at 226.06 50.8 0)
-			(effects
-				(font
-					(size 1.27 1.27)
-				)
-				(hide yes)
-			)
-		)
-		(property "PACKAGE" "None"
-			(at 226.06 50.8 0)
-			(effects
-				(font
-					(size 1.27 1.27)
-				)
-				(justify bottom)
-				(hide yes)
-			)
-		)
-		(property "PRICE" "$0.58 USD"
-			(at 226.06 50.8 0)
-			(effects
-				(font
-					(size 1.27 1.27)
-				)
-				(justify bottom)
-				(hide yes)
-			)
-		)
-		(property "MF" "Molex"
-			(at 226.06 50.8 0)
-			(effects
-				(font
-					(size 1.27 1.27)
-				)
-				(justify bottom)
-				(hide yes)
-			)
-		)
-		(property "AVAILABILITY" "Good"
-			(at 226.06 50.8 0)
-			(effects
-				(font
-					(size 1.27 1.27)
-				)
-				(justify bottom)
-				(hide yes)
-			)
-		)
-		(property "MP" "52271-0679"
-			(at 226.06 50.8 0)
-			(effects
-				(font
-					(size 1.27 1.27)
-				)
-				(justify bottom)
-				(hide yes)
-			)
-		)
-		(pin "1"
-		)
-		(pin "5"
-		)
-		(pin "4"
-		)
-		(pin "6"
-		)
-		(pin "3"
-		)
-		(pin "2"
-		)
-		(instances
-			(project "Raspi_Zero_TFT_Interface"
-				(path "/9fcf58ec-9ad6-40d8-a93b-d0fc15c15838"
-					(reference "CN6")
-					(unit 1)
-				)
-			)
-		)
-	)
-	(symbol
 		(lib_id "power:GND")
 		(at 246.38 121.92 0)
@@
 	)
 	(symbol
+		(lib_id "2024-10-22_14-40-48:522070860")
+		(at 233.68 45.72 0)
+		(mirror y)
+		(unit 1)
+		(exclude_from_sim no)
+		(in_bom yes)
+		(on_board yes)
+		(dnp no)
+		(fields_autoplaced yes)
+		(property "Reference" "J1"
+			(at 224.79 38.1 0)
+			(effects
+				(font
+					(size 1.524 1.524)
+				)
+			)
+		)
+		(property "Value" "522070860"
+			(at 224.79 40.64 0)
+			(effects
+				(font
+					(size 1.524 1.524)
+				)
+			)
+		)
+		(property "Footprint" "GenIILibrary:CON_522070860_MOL"
+			(at 247.396 43.18 0)
+			(effects
+				(font
+					(size 1.27 1.27)
+					(italic yes)
+				)
+				(hide yes)
+			)
+		)
+		(property "Datasheet" "522070860"
+			(at 233.68 45.72 0)
+			(effects
+				(font
+					(size 1.27 1.27)
+					(italic yes)
+				)
+				(hide yes)
+			)
+		)
+		(property "Description" ""
+			(at 233.68 45.72 0)
+			(effects
+				(font
+					(size 1.27 1.27)
+				)
+				(hide yes)
+			)
+		)
+		(pin "1"
+		)
+		(pin "5"
+		)
+		(pin "P1"
+		)
+		(pin "2"
+		)
+		(pin "3"
+		)
+		(pin "6"
+		)
+		(pin "8"
+		)
+		(pin "7"
+		)
+		(pin "P2"
+		)
+		(pin "4"
+		)
+		(instances
+			(project ""
+				(path "/9fcf58ec-9ad6-40d8-a93b-d0fc15c15838"
+					(reference "J1")
+					(unit 1)
+				)
+			)
+		)
+	)
+	(symbol
 		(lib_id "Device:C_Small")
 		(at 78.74 118.11 0)
@@
 			)
 		)
+		(pin "~{CHARGE_EN}" input
+			(at 193.04 129.54 180)
+			(effects
+				(font
+					(size 1.27 1.27)
+				)
+				(justify left)
+			)
+		)
