File: Raspi_Zero_TFT_Interface/Raspi_Zero_TFT_Interface.kicad_pcb (KiCad board)
At the start: 4 copper layers, 34 parts, among them CN1 USB_C_Receptacle_PowerOnly_6P, CN2 B2PS-VH, CN3 Molex FPC 541044031, CN4 Molex FPC 52271-0679, CN5 Conn_02x20_Odd_Even, CN6 Molex FPC 52271-0679, Q3 DMG3406L-7, Q4 SSM3J358R, SW2 Rocker Switch SPST, U1 AP5725WG-7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

Commit message: First draft layout of power pi board
Parts:
- added D10: LED, Diode_THT:D_T-1_P2.54mm_Vertical_AnodeUp, F.Cu at (62.9, 24.4)
- added D7: LED, Diode_THT:D_T-1_P2.54mm_Vertical_AnodeUp, F.Cu at (60.5, 28.0)
- C11, C19, C2, C20, C23, C24, C25, C26, C3, D1, D6, D8, L1, Q3, Q4, R14, R17, R18, R20, Rfb1, U1, U11, U13, U8: moved to F.Cu
- CN2: value B2PS-VH -> B2B-XH-A; footprint Connector_JST:JST_VH_B2P-VH_1x02_P3.96mm_Vertical -> Connector_JST:JST_XH_B2B-XH-A_1x02_P2.50mm_Vertical; moved to B.Cu
- CN3, CN4, CN6: moved to B.Cu
- CN5: footprint Connector_Samtec_HLE_SMD:Samtec_HLE-120-02-xxx-DV-BE_2x20_P2.54mm_Horizontal -> Connector_PinHeader_2.54mm:PinHeader_2x20_P2.54mm_Vertical; moved to B.Cu
- moved D1 99.3 mm to (46.8, 11.0), turned to 0 degrees
- moved L1 94.6 mm to (46.2, 9.12), turned to 0 degrees
- moved U1 91.3 mm to (42.7, 12.1), turned to 0 degrees
- moved C2 90.7 mm to (47.2, 12.8), turned to 0 degrees
- moved C3 86.0 mm to (42.4, 9.14)
- moved Rfb1 83.3 mm to (39.2, 12.2), turned to -90 degrees
- moved U13 77.3 mm to (54.1, 14.6), turned to 0 degrees
- moved R17 70.7 mm to (57.0, 27.9), turned to 0 degrees
- moved R20 70.1 mm to (57.1, 24.4), turned to 0 degrees
- moved C26 67.4 mm to (54.1, 19.2)
- moved C25 64.4 mm to (54.2, 11.9)
- moved C23 63.8 mm to (54.2, 10.1), turned to 0 degrees
- moved C24 63.1 mm to (54.1, 17.5)
- moved C11 48.0 mm to (10.8, 22.6), turned to 0 degrees
- moved Q3 47.4 mm to (10.6, 15.0), turned to 90 degrees
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Connections:
- C24 pad 1: /3V3 -> /3V3_Main
- C26 pad 1: /3V3 -> /3V3_Main
- CN3 pad 10: /GPIO25 -> /R5
- CN3 pad 11: /GPIO26 -> /R6
- CN3 pad 12: /GPIO27 -> /R7
- CN3 pad 4: /3V3 -> /3V3_Pi
- CN3 pad 6: /GPIO21 -> /R1
- CN3 pad 9: /GPIO24 -> /R4
- CN4 pad 1: /3V3 -> /3V3_Pi
- CN4 pad 3: /GPIO3 -> /SCL
- CN4 pad 4: /GPIO2 -> /SDA
- CN4 pad 5: /GPIO4 -> /~{INT}
- CN4 pad 6: /3V3 -> /3V3_Pi
- CN5 pad 1: /3V3 -> /Vcc
- CN5 pad 10: /GPIO15 -> GND
- CN5 pad 11: /G5 -> /G6
- CN5 pad 12: /G6 -> /G5
- CN5 pad 13: /GPIO27 -> GND
- CN5 pad 14: GND -> /R7
- CN5 pad 15: /G2 -> /G3
- CN5 pad 16: /G3 -> /G2
- CN5 pad 17: /3V3 -> /R4
- CN5 pad 18: /GPIO24 -> /3V3_Pi
- CN5 pad 19: /B6 -> GND
- CN5 pad 2: /Vcc -> /3V3_Pi
- CN5 pad 20: GND -> /B6
- CN5 pad 21: /B5 -> /R5
- CN5 pad 22: /GPIO25 -> /B5
- CN5 pad 23: /B7 -> /B4
- CN5 pad 24: /B4 -> /B7
- CN5 pad 25: GND -> /B3
- CN5 pad 26: /B3 -> GND
- CN5 pad 27: /CLK -> /DE
- CN5 pad 28: /DE -> /CLK
- CN5 pad 29: /B1 -> GND
- CN5 pad 3: /GPIO2 -> /Vcc
- CN5 pad 30: GND -> /B1
- CN5 pad 31: /B2 -> /PWM_EN
- CN5 pad 32: /G0 -> /B2
- CN5 pad 33: /G1 -> GND
- CN5 pad 34: GND -> /G1
- CN5 pad 35: /G7 -> /G4
- CN5 pad 36: /G4 -> /G7
- CN5 pad 37: /GPIO26 -> /DISP
- CN5 pad 38: /DISP -> /R6
- CN5 pad 39: GND -> /R1
- CN5 pad 4: /Vcc -> /SDA
- CN5 pad 40: /GPIO21 -> GND
- CN5 pad 5: /GPIO3 -> GND
- CN5 pad 6: GND -> /SCL
- CN5 pad 7: /GPIO4 -> /UART_TX
- CN5 pad 8: /GPIO14 -> /~{INT}
- CN5 pad 9: GND -> /UART_RX
- CN6 pad 3: /GPIO14 -> /UART_TX
- CN6 pad 4: /GPIO15 -> /UART_RX
- CN6 pad 6: /3V3 -> /3V3_Main
- U13 pad 4: /3V3 -> /3V3_Main
Routing:
- net /Power_Management_Minimal/5V_USB: track 0.00 -> 78.3 mm, vias 0 -> 2
- net /Vcc: track 0.00 -> 77.9 mm, vias 0 -> 2
- net /3V3_Pi: track 0.00 -> 67.6 mm, vias 0 -> 2
- net /~{INT}: track 0.00 -> 65.0 mm, vias 0 -> 3
- net /SCL: track 0.00 -> 60.9 mm, vias 0 -> 1
- net /UART_TX: track 0.00 -> 60.5 mm, vias 0 -> 2
- net /SDA: track 0.00 -> 58.9 mm, vias 0 -> 1
- net /UART_RX: track 0.00 -> 57.9 mm, vias 0 -> 2
- net /DISP: track 0.00 -> 50.6 mm, vias 0 -> 1
- net Net-(U11-STAT): track 0.00 -> 50.0 mm
- net /DE: track 0.00 -> 45.1 mm, vias 0 -> 1
- net GND: track 0.00 -> 45.0 mm, vias 0 -> 24
- net /G4: track 0.00 -> 39.6 mm, vias 0 -> 3
- net /R1: track 0.00 -> 32.7 mm
- net /R6: track 0.00 -> 32.1 mm, vias 0 -> 4
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- added copper zone on In2.Cu, net GND

Commit message: Completed (unflipped) board
Parts:
- added R3: 10k, Resistor_SMD:R_0603_1608Metric_Pad0.98x0.95mm_HandSolder, B.Cu at (3.00, 3.00)
- moved D7 62.1 mm to (1.91, 7.50)
- moved SW2 60.0 mm to (62.5, 2.23), turned to 0 degrees
- moved R17 59.3 mm to (2.59, 4.50), turned to 180 degrees
- moved C21 1.05 mm to (5.00, 3.00), turned to -90 degrees
Connections:
- D8 pad 1: Net-(D8-K) -> /Vcc
- Q4 pad 2: Net-(D8-K) -> /Vcc
- SW2 pad 1: Net-(D8-K) -> /Vcc
- SW2 pad 2: /Vcc -> Net-(SW2-B)
- U13 pad 1: /Vcc -> Net-(SW2-B)
Routing:
- net /Power_Management_Minimal/5V_USB: track 78.3 -> 23.5 mm, vias 2 -> 1
- net Net-(U11-STAT): track 50.0 -> 22.6 mm, vias 0 -> 2
- net /Vcc: track 77.9 -> 99.4 mm, vias 2 -> 5
- net Net-(SW2-B): track 0.00 -> 18.1 mm, vias 0 -> 1
- net Net-(D8-K): track 17.1 -> 0.00 mm, vias 2 -> 0
- net GND: track 45.0 -> 47.4 mm, vias 24 -> 39
- net /3V3_Pi: track 67.6 -> 65.5 mm
- net /DE: track 45.1 -> 46.4 mm
- net /B4: track 23.5 -> 24.5 mm
- net /B6: track 18.3 -> 18.9 mm
- net /UART_TX: track 60.5 -> 61.1 mm
- net Net-(D7-K): track 2.57 -> 3.10 mm
- net Net-(U13-PG): track 15.6 -> 15.3 mm, vias 0 -> 2
- net /R7: track 17.4 -> 17.6 mm, vias 2 -> 1
- added copper zone on F.Cu, net GND

Commit message: Partial Update
Connections:
- CN3 pad 1: /LED- -> unconnected-(CN3-Pad1)
- CN3 pad 10: /R5 -> GND
- CN3 pad 11: /R6 -> GND
- CN3 pad 12: /R7 -> /DISP
- CN3 pad 13: /G0 -> /CLK
- CN3 pad 14: /G1 -> GND
- CN3 pad 15: /G2 -> /B7
- CN3 pad 16: /G3 -> /B6
- CN3 pad 17: /G4 -> /B5
- CN3 pad 18: /G5 -> /B4
- CN3 pad 19: /G6 -> /B3
- CN3 pad 2: /LED+ -> unconnected-(CN3-Pad2)
- CN3 pad 20: /G7 -> /B2
- CN3 pad 21: /B0 -> /B1
- CN3 pad 22: /B1 -> /B0
- CN3 pad 23: /B2 -> /G7
- CN3 pad 24: /B3 -> /G6
- CN3 pad 25: /B4 -> /G5
- CN3 pad 26: /B5 -> /G4
- CN3 pad 27: /B6 -> /G3
- CN3 pad 28: /B7 -> /G2
- CN3 pad 29: GND -> /G1
- CN3 pad 3: GND -> unconnected-(CN3-Pad3)
- CN3 pad 30: /CLK -> /G0
- CN3 pad 31: /DISP -> /R7
- CN3 pad 32: GND -> /R6
- CN3 pad 33: GND -> /R5
- CN3 pad 34: /DE -> /R4
- CN3 pad 35: unconnected-(CN3-Pad35) -> /G3
- CN3 pad 36: GND -> /G2
- CN3 pad 37: unconnected-(CN3-Pad37) -> /R1
- CN3 pad 38: unconnected-(CN3-Pad38) -> /R0
- CN3 pad 39: unconnected-(CN3-Pad39) -> /3V3_Pi
- CN3 pad 4: /3V3_Pi -> unconnected-(CN3-Pad4)
- CN3 pad 40: unconnected-(CN3-Pad40) -> GND
- CN3 pad 5: /R0 -> unconnected-(CN3-Pad5)
- CN3 pad 6: /R1 -> unconnected-(CN3-Pad6)
- CN3 pad 7: /G2 -> GND
- CN3 pad 8: /G3 -> unconnected-(CN3-Pad8)
- CN3 pad 9: /R4 -> /DE
- CN3 pad P1: unconnected-(CN3-PadP1) -> /LED+
- CN3 pad P2: unconnected-(CN3-PadP2) -> /LED-
- CN4 pad 2: GND -> /~{INT}
- CN4 pad 3: /SCL -> /SDA
- CN4 pad 4: /SDA -> /SCL
- CN4 pad 5: /~{INT} -> GND
Routing:
- net /G4: track 39.7 -> 17.7 mm, vias 3 -> 1
- net /DE: track 46.4 -> 27.7 mm
- net /R4: track 19.8 -> 35.8 mm, vias 1 -> 0
- net /B5: track 20.0 -> 31.4 mm, vias 2 -> 3
- net /LED+: track 20.1 -> 10.5 mm, vias 1 -> 0
- net /G3: track 28.3 -> 20.3 mm
- net /R6: track 32.1 -> 24.2 mm, vias 4 -> 3
- net /G2: track 24.0 -> 17.0 mm, vias 4 -> 2
- net /R1: track 32.7 -> 27.5 mm
- net /R5: track 19.4 -> 14.4 mm
- net /LED-: track 10.6 -> 6.14 mm
- net /G1: track 28.1 -> 24.4 mm, vias 2 -> 1
- net /~{INT}: track 65.0 -> 62.8 mm, vias 3 -> 1
- net /SDA: track 58.9 -> 60.8 mm, vias 1 -> 3
- net /3V3_Pi: track 65.5 -> 63.8 mm
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
Commit message: Finalized Ras_Pi Power Board
Parts:
- added C1: 1uF, Capacitor_SMD:C_0603_1608Metric_Pad1.08x0.95mm_HandSolder, F.Cu at (19.4, 23.8)
- moved D1 5.21 mm to (41.7, 11.7)
- moved L1 5.21 mm to (41.0, 9.77)
- moved C2 5.21 mm to (42.1, 13.4)
- moved C3 5.21 mm to (37.2, 9.80)
- moved Rfb1 5.21 mm to (34.0, 12.9)
- moved U1 5.21 mm to (37.5, 12.7)
- moved D10 0.55 mm to (62.9, 24.9)
- moved R20 0.55 mm to (57.1, 24.9)
Connections:
- CN3 pad 10: GND -> /DISP
- CN3 pad 11: GND -> /CLK
- CN3 pad 12: /DISP -> GND
- CN3 pad 13: /CLK -> /B7
- CN3 pad 14: GND -> /B6
- CN3 pad 15: /B7 -> /B5
- CN3 pad 16: /B6 -> /B4
- CN3 pad 17: /B5 -> /B3
- CN3 pad 18: /B4 -> /B2
- CN3 pad 19: /B3 -> /B1
- CN3 pad 20: /B2 -> /B0
- CN3 pad 21: /B1 -> /G7
- CN3 pad 22: /B0 -> /G6
- CN3 pad 23: /G7 -> /G5
- CN3 pad 24: /G6 -> /G4
- CN3 pad 25: /G5 -> /G3
- CN3 pad 26: /G4 -> /G2
- CN3 pad 27: /G3 -> /G1
- CN3 pad 28: /G2 -> /G0
- CN3 pad 29: /G1 -> /R7
- CN3 pad 30: /G0 -> /R6
- CN3 pad 31: /R7 -> /R5
- CN3 pad 32: /R6 -> /R4
- CN3 pad 33: /R5 -> /G3
- CN3 pad 34: /R4 -> /G2
- CN3 pad 35: /G3 -> /R1
- CN3 pad 36: /G2 -> /R0
- CN3 pad 37: /R1 -> /3V3_Pi
- CN3 pad 38: /R0 -> GND
- CN3 pad 39: /3V3_Pi -> /LED+
- CN3 pad 40: GND -> /LED-
- CN3 pad 5: unconnected-(CN3-Pad5) -> GND
- CN3 pad 7: GND -> /DE
- CN3 pad 8: unconnected-(CN3-Pad8) -> GND
- CN3 pad 9: /DE -> GND
- CN3 pad P1: /LED+ -> unconnected-(CN3-PadP1)
- CN3 pad P2: /LED- -> unconnected-(CN3-PadP2)
Routing:
- net /LED+: track 10.5 -> 35.9 mm, vias 0 -> 1
- net /G4: track 17.7 -> 39.1 mm, vias 1 -> 2
- net /R1: track 27.5 -> 47.7 mm, vias 0 -> 2
- net /LED-: track 6.14 -> 26.0 mm
- net /DISP: track 50.6 -> 31.9 mm, vias 1 -> 2
- net /3V3_Pi: track 63.8 -> 80.5 mm, vias 2 -> 3
- net /R6: track 24.2 -> 40.9 mm, vias 3 -> 2
- net /G1: track 24.4 -> 37.2 mm, vias 1 -> 2
- net /B5: track 31.4 -> 18.8 mm, vias 3 -> 2
- net /R4: track 35.8 -> 24.1 mm, vias 0 -> 2
- net /R5: track 14.4 -> 26.0 mm, vias 1 -> 2
- net /CLK: track 28.9 -> 19.1 mm
- net /G2: track 17.0 -> 26.4 mm, vias 2 -> 3
- net /G7: track 31.9 -> 41.1 mm, vias 0 -> 1
- net /B7: track 25.2 -> 17.5 mm, vias 1 -> 0
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
Commit message: Small change to Raspi Board
Connections:
- C21 pad 1: /Vcc -> Net-(D8-K)
- D8 pad 1: /Vcc -> Net-(D8-K)
- Q4 pad 2: /Vcc -> Net-(D8-K)
- R3 pad 1: /Vcc -> Net-(D8-K)
- SW2 pad 2: Net-(SW2-B) -> Net-(D8-K)
- U13 pad 1: Net-(SW2-B) -> /Vcc
- U13 pad 7: (no net) -> GND
Routing:
- net Net-(D8-K): track 0.00 -> 79.9 mm, vias 0 -> 3
- net Net-(SW2-B): track 19.4 -> 0.00 mm, vias 1 -> 0
- net /Vcc: track 100.2 -> 90.6 mm, vias 5 -> 3
- net GND: track 45.1 -> 48.2 mm, vias 52 -> 51

Commit message: Nearly Finalized Boards
Parts:
- removed C21: 10u, Capacitor_SMD:C_0603_1608Metric_Pad1.08x0.95mm_HandSolder
- removed CN6: Molex FPC 52271-0679, GenIILibrary:MOLEX_52271-0679
- removed R3: 10k, Resistor_SMD:R_0603_1608Metric_Pad0.98x0.95mm_HandSolder
- removed U13: LD39050, Package_DFN_QFN:DFN-6-1EP_3x3mm_P0.95mm_EP1.7x2.6mm
- added C4: 22u, Capacitor_SMD:C_0603_1608Metric_Pad1.08x0.95mm_HandSolder, F.Cu at (57.5, 8.38)
- added J1: 522070860, GenIILibrary:CON_522070860_MOL, B.Cu at (62.6, 15.0)
- added Q1: SI2347DS-TI-GE3CT, Package_TO_SOT_SMD:SOT-23-3, B.Cu at (13.2, 14.8)
- added RPU1: 5k, Resistor_SMD:R_0603_1608Metric_Pad0.98x0.95mm_HandSolder, B.Cu at (16.4, 15.2)
- added U2: LD39200, Package_DFN_QFN:DFN-6-1EP_3x3mm_P0.95mm_EP1.7x2.6mm, F.Cu at (53.9, 12.8)
- C19: moved to B.Cu
- D8: value MSS1P3L -> PMEG3030EP,115; footprint Diode_SMD:D_MicroSMP_AK -> Diode_SMD:D_SOD-128
- moved SW2 58.6 mm to (3.90, 2.35), turned to -90 degrees
- moved CN1 8.00 mm to (-4.60, 24.7)
- moved D8 7.50 mm to (3.95, 14.4), turned to -90 degrees
- moved D7 7.43 mm to (-3.25, 2.16), turned to -90 degrees
- moved CN2 6.55 mm to (-2.90, 15.6), turned to 90 degrees
- moved C20 6.10 mm to (-0.07, 14.4)
- moved D6 5.62 mm to (5.95, 24.8), turned to -90 degrees
- moved C19 5.40 mm to (11.6, 11.0), turned to -90 degrees
- moved R14 4.34 mm to (17.8, 10.3), turned to -90 degrees
- moved C25 2.45 mm to (52.6, 10.0)
- moved Q4 2.35 mm to (8.47, 9.59), turned to 180 degrees
- moved C23 2.34 mm to (52.6, 8.40)
- moved Q3 2.18 mm to (8.55, 15.7), turned to 180 degrees
- moved C26 1.81 mm to (53.7, 17.4), turned to 0 degrees
- moved C24 1.81 mm to (53.7, 15.7), turned to 0 degrees
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Connections:
- C19 pad 2: /Power_Management_Minimal/5V_USB -> Net-(D7-A)
- C20 pad 1: /Power_Management_Minimal/V_Batt+ -> /V_Batt
- CN2 pad 1: /Power_Management_Minimal/V_Batt+ -> GND
- CN2 pad 2: GND -> /V_Batt
- D7 pad 2: /Power_Management_Minimal/5V_USB -> Net-(D7-A)
- Q4 pad 2: Net-(D8-K) -> /V_Batt
- Q4 pad 3: /Power_Management_Minimal/V_Batt+ -> Net-(D8-K)
- U11 pad 3: /Power_Management_Minimal/V_Batt+ -> /V_Batt
- U11 pad 4: /Power_Management_Minimal/5V_USB -> Net-(D7-A)
Routing:
- net /V_Batt: track 0.00 -> 98.9 mm, vias 0 -> 1
- net /~{CHARGE_EN}: track 0.00 -> 68.0 mm, vias 0 -> 3
- net Net-(D8-K): track 79.9 -> 16.5 mm, vias 3 -> 1
- net Net-(D7-A): track 0.00 -> 22.8 mm, vias 0 -> 1
- net /Power_Management_Minimal/V_Batt+: track 16.8 -> 0.00 mm, vias 2 -> 0
- net /Vcc: track 90.6 -> 78.4 mm, vias 3 -> 2
- net Net-(U11-STAT): track 22.6 -> 13.0 mm, vias 2 -> 0
- net /Power_Management_Minimal/5V_USB: track 23.4 -> 17.3 mm
- net Net-(U2-PWRGD): track 15.4 -> 20.4 mm
- net /3V3_Main: track 7.86 -> 12.8 mm
- net Net-(D7-K): track 3.10 -> 7.50 mm
- net /USB_VCC2: track 2.83 -> 6.02 mm
- net /USB_VCC1: track 2.95 -> 5.30 mm
- net /Power_Management_Minimal/VBus: track 22.3 -> 23.6 mm
- net /UART_RX: track 57.9 -> 56.9 mm
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
Commit message: Final commit before order
Changed lines of the file:
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@@
 		)
 		(property "Value" "100n"
-			(at 0 1.43 360)
+			(at 0 1.43 0)
 			(layer "F.Fab")
 			(hide yes)
@@
 		)
 		(fp_text user "${REFERENCE}"
-			(at 0 0 360)
+			(at 0 0 0)
 			(layer "F.Fab")
 			(hide yes)
@@
 		)
 		(property "Value" "1uF/XR5"
-			(at 0 1.43 360)
+			(at 0 1.43 0)
 			(layer "F.Fab")
 			(hide yes)
@@
 		)
 		(fp_text user "${REFERENCE}"
-			(at 0 0 360)
+			(at 0 0 0)
 			(layer "F.Fab")
 			(hide yes)
@@
 		)
 		(fill none)
-		(layer "Dwgs.User")
+		(layer "F.SilkS")
 	)
 	(segment
