File: FrontEndPrototype_Rev2_Heater/FrontEndPrototype_Rev2_Heater.kicad_sch (KiCad schematic)
At the start: 16 parts, among them J1 Conn_01x02_Pin, J2 Conn_01x02_Pin, J3 Conn_01x02_Pin, J4 Conn_01x02_Pin

Commit message: Boards nearly finalized
Parts:
- removed R1, R2, R3, R4, R5, R6, R7, R8: 50, Resistor_SMD:R_2512_6332Metric_Pad1.40x3.35mm_HandSolder, symbol Device:R_Small_US
- added H1, H10, H11, H12, H13, H14, H15, H16, H2, H3, H4, H5, H6, H7, H8, H9: PogoPinClearanceHole, GenIILibrary:PogoClearanceHole, symbol Mechanical:MountingHole
- added J5, J6, J7, J8: Conn_01x02_Pin, GenIILibrary:Samtec_Pin_Socket_SS_102_G_2, symbol Connector:Conn_01x02_Pin
- added R10, R11, R12, R13, R14, R15, R16, R9: 50, Resistor_SMD:R_2010_5025Metric_Pad1.40x2.65mm_HandSolder, symbol Device:R_Small_US
- added TH5, TH6, TH7, TH8: Thermistor_NTC, Resistor_SMD:R_0603_1608Metric_Pad0.98x0.95mm_HandSolder, symbol Device:Thermistor_NTC
Connections:
- net Vdd_Heater is gone; now on net Vdd_Heater_1: J1.1 (Pin_1), TH1.1, TH2.1, TH3.2, TH4.2
- net Vdd_Heater_1: now reaches J3.1 (Pin_1)
- net GND renamed GND_1
- new net: J7.1 (Pin_1), TH5.2
- new net: J7.2 (Pin_2), TH6.1
- new net: J8.1 (Pin_1), TH7.2
- new net: J8.2 (Pin_2), TH8.1
- new net GND_2: J5.2 (Pin_2), J6.2 (Pin_2)
- new net HGND: J6.1 (Pin_1), R10.1, R11.1, R12.1, R13.1, R14.1, R15.1, R16.1, R9.1
- new net Vdd_Heater_2: J5.1 (Pin_1), R10.2, R11.2, R12.2, R13.2, R14.2, R15.2, R16.2, R9.2, TH5.1, TH6.2, TH7.1, TH8.2
Other:
- note added: "Type I: Trace Element"
- note added: "Type II: Discrete Resistors"
- moved on the sheet: J1, J2, J3, J4, TH1, TH2, TH3, TH4

Commit message: Nearly Finalized Boards
Parts:
- removed H1, H2, H3, H4, H5, H6, H7, H8: PogoPinClearanceHole, GenIILibrary:PogoClearanceHole, symbol Mechanical:MountingHole
- removed J2, J3, J4, J8: Conn_01x02_Pin, GenIILibrary:Samtec_Pin_Socket_SS_102_G_2, symbol Connector:Conn_01x02_Pin
- removed TH1, TH2, TH3, TH4, TH6, TH8: Thermistor_NTC, Resistor_SMD:R_0603_1608Metric_Pad0.98x0.95mm_HandSolder, symbol Device:Thermistor_NTC
Connections:
- net Vdd_Heater_1 is gone; now on net Vdd_Heater_2: J1.1 (Pin_1)
- net Vdd_Heater_2: no longer TH5.1, TH7.1
- net at J7.1 (Pin_1): now also TH5.1; no longer TH5.2
- net at J7.2 (Pin_2): now also TH5.2
- net at TH7.2: now also J6.2 (Pin_2)
- net GND_1: no longer names the net of J1.2 (Pin_2)
- net GND_1: now also J5.2 (Pin_2), R10.1, R11.1, R12.1, R13.1, R14.1, R15.1, R16.1, R9.1
- removed net GND_2: J5.2 (Pin_2), J6.2 (Pin_2)
- removed net HGND: J6.1 (Pin_1), R10.1, R11.1, R12.1, R13.1, R14.1, R15.1, R16.1, R9.1
- new net: J6.1 (Pin_1), TH7.1
Other:
- note removed: "Type I: Trace Element"
- moved on the sheet: J5, J6, TH5, TH7

Commit message: Final Edit Before Check and Combine
Parts:
- added J2, J3: Conn_01x02_Pin, GenIILibrary:Thermistor_ExtensionPad, symbol Connector:Conn_01x02_Pin
Connections:
- net at J7.1 (Pin_1), TH5.1: now also J2.1 (Pin_1)
- net at J7.2 (Pin_2), TH5.2: now also J2.2 (Pin_2)
- net at J6.1 (Pin_1), TH7.1: now also J3.1 (Pin_1)
- net at J6.2 (Pin_2), TH7.2: now also J3.2 (Pin_2)
Other:
- note added: "Extension Pads for Thermistor Connection"
Changed lines of the file:
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@@
 	(paper "A4")
+	(junction
+		(at 270.51 114.3)
+		(diameter 0)
+		(color 0 0 0 0)
+	)
 	(junction
 		(at 184.15 57.15)
@@
 	)
 	(junction
+		(at 267.97 116.84)
+		(diameter 0)
+		(color 0 0 0 0)
+	)
+	(junction
 		(at 246.38 46.99)
 		(diameter 0)
@@
 	)
 	(junction
+		(at 213.36 116.84)
+		(diameter 0)
+		(color 0 0 0 0)
+	)
+	(junction
+		(at 215.9 114.3)
+		(diameter 0)
+		(color 0 0 0 0)
+	)
+	(junction
 		(at 209.55 46.99)
 		(diameter 0)
@@
 	(wire
 		(pts
-			(xy 266.7 116.84) (xy 271.78 116.84)
+			(xy 266.7 116.84) (xy 267.97 116.84)
 		)
 		(stroke
@@
 	(wire
 		(pts
-			(xy 209.55 116.84) (xy 219.71 116.84)
+			(xy 209.55 116.84) (xy 213.36 116.84)
+		)
+		(stroke
+			(width 0)
+			(type default)
+		)
+	)
+	(wire
+		(pts
+			(xy 267.97 105.41) (xy 267.97 116.84)
 		)
 		(stroke
@@
 	(wire
 		(pts
-			(xy 209.55 114.3) (xy 219.71 114.3)
+			(xy 209.55 114.3) (xy 215.9 114.3)
 		)
 		(stroke
@@
 	(wire
 		(pts
+			(xy 270.51 105.41) (xy 270.51 114.3)
+		)
+		(stroke
+			(width 0)
+			(type default)
+		)
+	)
+	(wire
+		(pts
 			(xy 200.66 67.31) (xy 209.55 67.31)
 		)
@@
 	(wire
 		(pts
+			(xy 213.36 116.84) (xy 219.71 116.84)
+		)
+		(stroke
+			(width 0)
+			(type default)
+		)
+	)
+	(wire
+		(pts
 			(xy 200.66 46.99) (xy 200.66 54.61)
 		)
@@
 	(wire
 		(pts
+			(xy 215.9 114.3) (xy 219.71 114.3)
+		)
+		(stroke
+			(width 0)
+			(type default)
+		)
+	)
+	(wire
+		(pts
 			(xy 219.71 59.69) (xy 219.71 67.31)
 		)
@@
 	(wire
 		(pts
+			(xy 270.51 114.3) (xy 271.78 114.3)
+		)
+		(stroke
+			(width 0)
+			(type default)
+		)
+	)
+	(wire
+		(pts
 			(xy 184.15 57.15) (xy 184.15 46.99)
 		)
@@
 	(wire
 		(pts
+			(xy 215.9 106.68) (xy 215.9 114.3)
+		)
+		(stroke
+			(width 0)
+			(type default)
+		)
+	)
+	(wire
+		(pts
 			(xy 209.55 46.99) (xy 209.55 54.61)
 		)
@@
 	(wire
 		(pts
+			(xy 267.97 116.84) (xy 271.78 116.84)
+		)
+		(stroke
+			(width 0)
+			(type default)
+		)
+	)
+	(wire
+		(pts
 			(xy 177.8 57.15) (xy 184.15 57.15)
 		)
@@
 	(wire
 		(pts
-			(xy 266.7 114.3) (xy 271.78 114.3)
+			(xy 266.7 114.3) (xy 270.51 114.3)
 		)
 		(stroke
@@
 	(wire
 		(pts
+			(xy 213.36 106.68) (xy 213.36 116.84)
+		)
+		(stroke
+			(width 0)
+			(type default)
+		)
+	)
+	(wire
+		(pts
 			(xy 228.6 46.99) (xy 228.6 54.61)
 		)
@@
 			(width 0)
 			(type default)
+		)
+	)
+	(text "Extension Pads for Thermistor Connection"
+		(exclude_from_sim no)
+		(at 242.57 98.806 0)
+		(effects
+			(font
+				(size 1.27 1.27)
+			)
 		)
 	)
@@
 	(symbol
 		(lib_id "Connector:Conn_01x02_Pin")
+		(at 270.51 100.33 270)
+		(unit 1)
+		(exclude_from_sim no)
+		(in_bom yes)
+		(on_board yes)
+		(dnp no)
+		(property "Reference" "J3"
+			(at 275.59 100.965 0)
+			(effects
+				(font
+					(size 1.27 1.27)
+				)
+			)
+		)
+		(property "Value" "Conn_01x02_Pin"
+			(at 273.05 100.965 0)
+			(effects
+				(font
+					(size 1.27 1.27)
+				)
+				(hide yes)
+			)
+		)
+		(property "Footprint" "GenIILibrary:Thermistor_ExtensionPad"
+			(at 270.51 100.33 0)
+			(effects
+				(font
+					(size 1.27 1.27)
+				)
+				(hide yes)
+			)
+		)
+		(property "Datasheet" "~"
+			(at 270.51 100.33 0)
+			(effects
+				(font
+					(size 1.27 1.27)
+				)
+				(hide yes)
+			)
+		)
+		(property "Description" ""
+			(at 270.51 100.33 0)
+			(effects
+				(font
+					(size 1.27 1.27)
+				)
+				(hide yes)
+			)
+		)
+		(pin "1"
+		)
+		(pin "2"
+		)
+		(instances
+			(project "FrontEndPrototype_Rev2_Heater"
+				(path "/e436919c-dde8-4a59-b391-4407947ae518"
+					(reference "J3")
+					(unit 1)
+				)
+			)
+		)
+	)
+	(symbol
+		(lib_id "Connector:Conn_01x02_Pin")
 		(at 193.04 57.15 0)
 		(mirror y)
@@
 					(unit 1)
 				)
+			)
+		)
+	)
+	(symbol
+		(lib_id "Connector:Conn_01x02_Pin")
+		(at 215.9 101.6 270)
+		(unit 1)
+		(exclude_from_sim no)
+		(in_bom yes)
+		(on_board yes)
+		(dnp no)
+		(property "Reference" "J2"
+			(at 220.98 102.235 0)
+			(effects
+				(font
+					(size 1.27 1.27)
+				)
+			)
+		)
+		(property "Value" "Conn_01x02_Pin"
+			(at 218.44 102.235 0)
+			(effects
+				(font
+					(size 1.27 1.27)
+				)
+				(hide yes)
+			)
+		)
+		(property "Footprint" "GenIILibrary:Thermistor_ExtensionPad"
+			(at 215.9 101.6 0)
+			(effects
+				(font
+					(size 1.27 1.27)
+				)
+				(hide yes)
+			)
+		)
+		(property "Datasheet" "~"
+			(at 215.9 101.6 0)
+			(effects
+				(font
+					(size 1.27 1.27)
+				)
+				(hide yes)
+			)
+		)
+		(property "Description" ""
+			(at 215.9 101.6 0)
+			(effects
+				(font
+					(size 1.27 1.27)
+				)
+				(hide yes)
+			)
+		)
+		(pin "1"
+		)
+		(pin "2"
+		)
+		(instances
+			(project "FrontEndPrototype_Rev2_Heater"
+				(path "/e436919c-dde8-4a59-b391-4407947ae518"
+					(reference "J2")
+					(unit 1)
+				)
